Commit message: finished dynamic config for spawn multiple robots with different colors

File: xacro/barista_robot_model.urdf.xacro (robot description, xacro)
@@ -1,5 +1,4 @@
 <?xml version="1.0"?>
 <robot xmlns:xacro="http://www.ros.org/wiki/xacro" name="barista_bot">
-<xacro:property name="robot_name" value="$(arg robot_name)"/>
 <xacro:include filename="$(find barista_robot_description)/xacro/caster_wheel.xacro" />
 <xacro:include filename="$(find barista_robot_description)/xacro/cup_holder_tray.xacro" />
@@ -7,5 +6,10 @@
 <xacro:include filename="$(find barista_robot_description)/xacro/laser_scanner.xacro" />
 <xacro:include filename="$(find barista_robot_description)/xacro/standoff_rod.xacro" />
+<xacro:arg name="robot_name" default="barista_bot"/>
 <xacro:arg name="include_laser" default="true"/>
+<xacro:arg name="gazebo_color" default="Gazebo/White"/>
+<xacro:property name="robot_name" value="$(arg robot_name)"/>
+<xacro:property name="gazebo_color" value="$(arg gazebo_color)"/>
+<xacro:property name="include_laser" value="$(arg include_laser)"/>
 <material name="blue">
       <color rgba="0.0 0.0 1.0 1"/>
@@ -50,5 +54,5 @@
 </joint>
 <gazebo reference="main_body_link">
-    <material>Gazebo/Blue</material>
+    <material>${gazebo_color}</material>
 </gazebo>
 <!--Standoff Rods-->
@@ -106,5 +110,5 @@
 </joint>
 <!--Cup Holder Tray-->
-<xacro:cup_holder_tray />
+<xacro:cup_holder_tray color="${gazebo_color}" />
 <joint name="main_body_to_cup_holder_link_joint" type="fixed">
     <origin rpy="0 0 0" xyz="0 0 0.3425" />
@@ -148,5 +152,5 @@
 </gazebo>
 <!--Laser-->
-<xacro:if value="$(arg include_laser)">
+<xacro:if value="${include_laser}">
     <xacro:laser_scanner />
     <joint name="laser_scan_link_joint" type="fixed">
@@ -179,5 +183,5 @@
             <ros>
                 <namespace>/${robot_name}</namespace>
-                <remapping>~/out:=/scan</remapping>
+                <remapping>~/out:=scan</remapping>
             </ros>
             <output_type>sensor_msgs/LaserScan</output_type>

File: xacro/cup_holder_tray.xacro (robot description, xacro)
@@ -1,5 +1,5 @@
 <?xml version="1.0"?>
 <robot xmlns:xacro="http://www.ros.org/wiki/xacro" name="barista_bot">
-<xacro:macro name="cup_holder_tray">
+<xacro:macro name="cup_holder_tray" params="color">
     <link name="cup_holder_link">
         <visual>
@@ -21,5 +21,5 @@
     </link>
     <gazebo reference="cup_holder_link">
-        <material>Gazebo/Blue</material>
+        <material>${color}</material>
     </gazebo>
 </xacro:macro>

Commit message: Added multi robot view for rviz

File: xacro/barista_robot_model.urdf.xacro (robot description, xacro)
@@ -9,6 +9,8 @@
 <xacro:arg name="include_laser" default="true"/>
 <xacro:arg name="gazebo_color" default="Gazebo/White"/>
+<xacro:arg name="color" default="White"/>
 <xacro:property name="robot_name" value="$(arg robot_name)"/>
 <xacro:property name="gazebo_color" value="$(arg gazebo_color)"/>
+<xacro:property name="color" value="$(arg color)"/>
 <xacro:property name="include_laser" value="$(arg include_laser)"/>
 <material name="blue">
@@ -35,5 +37,5 @@
             <cylinder length="0.155" radius="0.178" />
         </geometry>
-        <material name="blue" />
+        <material name="${color}" />
     </visual>
     <collision>
@@ -110,5 +112,5 @@
 </joint>
 <!--Cup Holder Tray-->
-<xacro:cup_holder_tray color="${gazebo_color}" />
+<xacro:cup_holder_tray gazebo_color="${gazebo_color}" color="${color}"/>
 <joint name="main_body_to_cup_holder_link_joint" type="fixed">
     <origin rpy="0 0 0" xyz="0 0 0.3425" />
@@ -147,6 +149,6 @@
         <publish_odom>true</publish_odom>
         <publish_odom_tf>true</publish_odom_tf>
-        <odometry_frame>odom</odometry_frame>
-        <robot_base_frame>base_link</robot_base_frame>
+        <odometry_frame>${robot_name}/odom</odometry_frame>
+        <robot_base_frame>${robot_name}/base_link</robot_base_frame>
     </plugin>
 </gazebo>

File: xacro/cup_holder_tray.xacro (robot description, xacro)
@@ -1,5 +1,5 @@
 <?xml version="1.0"?>
 <robot xmlns:xacro="http://www.ros.org/wiki/xacro" name="barista_bot">
-<xacro:macro name="cup_holder_tray" params="color">
+<xacro:macro name="cup_holder_tray" params="gazebo_color color">
     <link name="cup_holder_link">
         <visual>
@@ -7,5 +7,5 @@
                 <cylinder length=".090" radius="0.160" />
             </geometry>
-            <material name="blue"/>
+            <material name="${color}"/>
         </visual>
         <collision>
@@ -21,5 +21,5 @@
     </link>
     <gazebo reference="cup_holder_link">
-        <material>${color}</material>
+        <material>${gazebo_color}</material>
     </gazebo>
 </xacro:macro>
