Commit message: Second submission attempt

File: urdf/barista_robot_model.urdf (robot description, URDF)
Before this commit: robot barista_bot, 16 links, 15 joints
Links:
- removed link back_pitch_link
- removed link back_roll_link
- removed link back_yaw_link
- removed link front_pitch_link
- removed link front_roll_link
- removed link front_yaw_link
- added link back_caster_link, mass 0.01; collision sphere radius=0.0352; visual sphere radius=0.0352
- added link front_caster_link, mass 0.01; collision sphere radius=0.0352; visual sphere radius=0.0352
- link cup_holder_link: mass 0.25 -> 0.05
Joints:
- removed joint back_roll_to_front_pitch_joint
- removed joint back_yaw_to_front_roll_joint
- removed joint front_roll_to_front_pitch_joint
- removed joint front_yaw_to_front_roll_joint
- removed joint main_body_to_back_yaw_joint
- removed joint main_body_to_front_yaw_joint
- added joint main_body_to_back_caster_joint: type fixed, parent main_body_link, child back_caster_link, origin xyz=-0.125 0 -0.1 rpy=0 0 0
- added joint main_body_to_front_caster_joint: type fixed, parent main_body_link, child front_caster_link, origin xyz=0.125 0 -0.1 rpy=0 0 0
- joint base_link_joint: origin xyz=0 0 0.15 rpy=0 0 0 -> xyz=0 0 0.135 rpy=0 0 0
- joint main_body_to_left_wheel_link_joint: limit (none) -> effort=10000 velocity=1000
- joint main_body_to_right_wheel_link_joint: limit (none) -> effort=10000 velocity=1000

File: xacro/barista_robot_model.urdf.xacro (robot description, xacro)
@@ -44,5 +44,5 @@
 </link>
 <joint name="base_link_joint" type="fixed">
-    <origin rpy="0 0 0" xyz="0 0 0.15" />
+    <origin rpy="0 0 0" xyz="0 0 0.135" />
     <parent link="base_link" />
     <child link="main_body_link" />
@@ -95,18 +95,14 @@
 <xacro:caster_wheel position="back" />
 <joint name="main_body_to_front_caster_joint" type="continuous">
-    <origin rpy="0 0 0" xyz="0.120 0 -0.0878" />
-    <parent link="main_body_link" />
-    <child link="front_yaw_link" />
+    <origin rpy="0 0 0" xyz="0.125 0 -0.1" />
+    <parent link="main_body_link"/>
+    <child link="front_caster_link"/>
     <axis xyz="0 0 1" />
-    <limit effort="1000.0" velocity="100.0" />
-    <dynamics damping="0.0" friction="0.1"/>
 </joint>
-<joint name="main_body_to_back_yaw_joint" type="continuous">
-    <origin rpy="0 0 0" xyz="-0.120 0 -0.0878" />
-    <parent link="main_body_link" />
-    <child link="back_yaw_link" />
+<joint name="main_body_to_back_caster_joint" type="continuous">
+    <origin rpy="0 0 0" xyz="-0.125 0 -0.1" />
+    <parent link="main_body_link"/>
+    <child link="back_caster_link"/>
     <axis xyz="0 0 1" />
-    <limit effort="1000.0" velocity="100.0" />
-    <dynamics damping="0.0" friction="0.1"/>
 </joint>
 <!--Cup Holder Tray-->
@@ -127,10 +123,4 @@
     <joint_name>main_body_to_right_wheel_link_joint</joint_name>
     <joint_name>main_body_to_left_wheel_link_joint</joint_name>
-    <joint_name>main_body_to_front_yaw_joint</joint_name>
-    <joint_name>main_body_to_back_yaw_joint</joint_name>
-    <joint_name>front_yaw_to_front_roll_joint</joint_name>
-    <joint_name>front_roll_to_front_pitch_joint</joint_name>
-    <joint_name>back_yaw_to_front_roll_joint</joint_name>
-    <joint_name>back_roll_to_front_pitch_joint</joint_name>
 </plugin>
 </gazebo>
@@ -165,5 +155,5 @@
     <gazebo reference="laser_scan_link">
         <sensor name="sensor_ray" type="ray">
-            <pose>0 0 0 0 0 0</pose>
+            <pose>0 0 0.34 0 0 0</pose>
             <ray>
             <scan>

File: xacro/caster_wheel.xacro (robot description, xacro)
@@ -2,16 +2,15 @@
 <robot xmlns:xacro="http://www.ros.org/wiki/xacro" name="barista_bot">
 <xacro:macro name="caster_wheel" params="position">
-    <link name="${position}_yaw_link">
+    <!--Caster Wheel Front-->
+    <link name="${position}_caster_link">
         <visual>
-            <origin rpy="0 1.5707 1.5707" xyz="0 0 0"/>
             <geometry>
-                <cylinder length="0.0206" radius="0.0352"/>
+                <sphere radius="0.0352"/>
             </geometry>
-            <material name="green_light"/>
+            <material name="white"/>
         </visual>
         <collision>
-            <origin rpy="0 1.5707 1.5707" xyz="0 0 0"/>
             <geometry>
-            <cylinder length="0.0206" radius="0.0352"/>
+                <sphere radius="0.0352"/>
             </geometry>
         </collision>
@@ -19,75 +18,14 @@
             <mass value="0.01"/>
             <origin rpy="0 0 0" xyz="0 0 0"/>
-            <inertia ixx="0.0000034512333333" ixy="0" ixz="0" iyy=".0000034512333333" iyz="0" izz="0.0000061952"/>
+            <inertia ixx="0.00000495616" ixy="0" ixz="0" iyy="0.00000495616" iyz="0" izz="0.00000495616"/>
         </inertial>
     </link>
-    <gazebo reference="${position}_yaw_link">
-        <material>Gazebo/Green</material>
-    </gazebo>
-    <link name="${position}_roll_link">
-        <visual>
-            <origin rpy="0 1.5707 1.5707" xyz="0 0 0"/>
-            <geometry>
-                <cylinder length="0.0206" radius="0.0352"/>
-            </geometry>
-            <material name="red"/>
-        </visual>
-        <collision>
-            <origin rpy="0 1.5707 1.5707" xyz="0 0 0"/>
-            <geometry>
-            <cylinder length="0.0206" radius="0.0352"/>
-            </geometry>
-        </collision>
-        <inertial>
-            <mass value="0.01"/>
-            <origin rpy="0 0 0" xyz="0 0 0"/>
-            <inertia ixx="0.0000034512333333" ixy="0" ixz="0" iyy=".0000034512333333" iyz="0" izz="0.0000061952"/>
-        </inertial>
-    </link>
-    <joint name="${position}_yaw_to_roll_joint" type="continuous">
-        <origin rpy="0 0 0" xyz="0 0 0" />
-        <parent link="${position}_yaw_link" />
-        <child link="${position}_roll_link" />
-        <axis xyz="1 0 0" />
-        <limit effort="1000.0" velocity="100.0" />
-        <dynamics damping="0.0" friction="0.1"/>
-    </joint>
-    <gazebo reference="${position}_roll_link">
-        <material>Gazebo/Red</material>
-    </gazebo>
-    <link name="${position}_pitch_link">
-        <visual>
-            <origin rpy="0 1.5707 1.5707" xyz="0 0 0"/>
-            <geometry>
-                <sphere radius="0.0352"/>
-            </geometry>
-            <material name="black"/>
-        </visual>
-        <collision>
-            <geometry>
-            <sphere radius="0.0352"/>
-            </geometry>
-        </collision>
-        <inertial>
-        <mass value="0.01"/>
-        <origin rpy="0 0 0" xyz="0 0 0"/>
-        <inertia ixx="0.00000495616" ixy="0" ixz="0" iyy="0.00000495616" iyz="0" izz="0.00000495616"/>
-        </inertial>
-    </link>
-    <gazebo reference="${position}_pitch_link">
-        <kp>1000</kp>
+    <gazebo reference="${position}_caster_link">
+        <kp>1000000</kp>
         <kd>100</kd>
-        <mu1>0.01</mu1>
-        <mu2>0.01</mu2>
+        <mu1>0.0</mu1>
+        <mu2>0.0</mu2>
         <material>Gazebo/White</material>
     </gazebo>
-    <joint name="${position}_roll_to_pitch_joint" type="continuous">
-        <origin rpy="0 0 0" xyz="0 0 0" />
-        <parent link="${position}_roll_link" />
-        <child link="${position}_pitch_link" />
-        <axis xyz="0 1 0" />
-        <limit effort="1000.0" velocity="100.0" />
-        <dynamics damping="0.0" friction="0.1"/>
-    </joint>
 </xacro:macro>
 </robot>

File: xacro/cup_holder_tray.xacro (robot description, xacro)
@@ -15,7 +15,7 @@
         </collision>
         <inertial>
-        <mass value="0.25"/>
+        <mass value="0.05"/>
         <origin rpy="0 0 0" xyz="0 0 0"/>
-        <inertia ixx="0.00176875" ixy="0" ixz="0" iyy="0.00176875" iyz="0" izz="0.0032"/>
+        <inertia ixx="0.00035375" ixy="0" ixz="0" iyy="0.00035375" iyz="0" izz="0.00064"/>
         </inertial>
     </link>

File: xacro/drive_wheel.xacro (robot description, xacro)
@@ -24,4 +24,5 @@
     <gazebo reference="${link_name}">
         <kp>1000</kp>
+        <kp>10000000</kp>
         <kd>100</kd>
         <mu1>1.0</mu1>

Commit message: finished fixes from submission 2. Ready for submission 3

File: urdf/barista_robot_model.urdf (robot description, URDF)
Before this commit: robot barista_bot, 12 links, 11 joints
Links:
- added link laser_scan_frame
Joints:
- added joint laser_scan_frame_to_link_joint: type fixed, parent laser_scan_link, child laser_scan_frame, origin xyz=0 0 .055 rpy=0 0 0

File: xacro/barista_robot_model.urdf.xacro (robot description, xacro)
@@ -94,15 +94,13 @@
 <xacro:caster_wheel position="front" />
 <xacro:caster_wheel position="back" />
-<joint name="main_body_to_front_caster_joint" type="continuous">
+<joint name="main_body_to_front_caster_joint" type="fixed">
     <origin rpy="0 0 0" xyz="0.125 0 -0.1" />
     <parent link="main_body_link"/>
     <child link="front_caster_link"/>
-    <axis xyz="0 0 1" />
 </joint>
-<joint name="main_body_to_back_caster_joint" type="continuous">
+<joint name="main_body_to_back_caster_joint" type="fixed">
     <origin rpy="0 0 0" xyz="-0.125 0 -0.1" />
     <parent link="main_body_link"/>
     <child link="back_caster_link"/>
-    <axis xyz="0 0 1" />
 </joint>
 <!--Cup Holder Tray-->

Commit message: Final commit before first submission

File: urdf/barista_robot_model.urdf (robot description, URDF)
Before this commit: robot barista_bot, 13 links, 12 joints
Joints:
- joint main_body_to_left_wheel_link_joint: origin xyz=0 -0.148 -0.1 rpy=0 0 0 -> xyz=0 0.148 -0.1 rpy=0 0 0
- joint main_body_to_right_wheel_link_joint: origin xyz=0 0.148 -.1 rpy=0 0 0 -> xyz=0 -0.148 -.1 rpy=0 0 0

File: xacro/barista_robot_model.urdf.xacro (robot description, xacro)
@@ -87,5 +87,5 @@
 <xacro:drive_wheel link_name="left_wheel_link" wheel_radius="0.0352" wheel_width="0.0206" />
 <joint name="main_body_to_right_wheel_link_joint" type="continuous">
-    <origin rpy="0 0 0" xyz="0 0.148 -.1" />
+    <origin rpy="0 0 0" xyz="0 -0.148 -.1" />
     <parent link="main_body_link" />
     <child link="right_wheel_link" />
@@ -93,5 +93,5 @@
 </joint>
 <joint name="main_body_to_left_wheel_link_joint" type="continuous">
-    <origin rpy="0 0 0" xyz="0 -0.148 -0.1" />
+    <origin rpy="0 0 0" xyz="0 0.148 -0.1" />
     <parent link="main_body_link" />
     <child link="left_wheel_link" />
